Commit message: kuka movement implemented (height problem)

File: catkin_ws/src/air_hockey/urdf/new_kuka.urdf (robot description, URDF)
Before this commit: robot kuka_iiwa14, 13 links, 12 joints
Links:
- link mallet: geometry collision cylinder length=0.05 radius=0.05; visual cylinder length=0.05 radius=0.05

File: catkin_ws/src/air_hockey/urdf/puck.urdf (robot description, URDF)
Before this commit: robot air_hockey_puck, 1 links, 0 joints
Links:
- link puck: geometry collision cylinder length=0.020 radius=0.025; visual cylinder length=0.020 radius=0.025

Commit message: Random Changes

File: catkin_ws/src/air_hockey/urdf/new_kuka.urdf (robot description, URDF)
Before this commit: robot kuka_iiwa14, 13 links, 12 joints
Links:
- link ball_link_1: geometry visual sphere radius=0.03
- link pole: geometry visual cylinder length=0.4 radius=0.01
Joints:
- joint fixed_mallet_joint: origin xyz=0 0 0 rpy=0 0 0.03 -> xyz=0 0 0.05 rpy=0 0 0
